Commit message: revert to original urdf

File: plastic_description/urdf/plastic/plastic_macro.ros2_control.xacro (robot description, xacro)
@@ -12,8 +12,4 @@
     <ros2_control name="${name}" type="system">
       <hardware>
-        <!--change this after adding HI-->
-        <plugin>ros2_control_demo_example_2/DiffBotSystemHardware</plugin>
-        <param name="example_param_hw_start_duration_sec">0</param>
-        <param name="example_param_hw_stop_duration_sec">3.0</param>
         <xacro:if value="${use_mock_hardware}">
           <plugin>mock_components/GenericSystem</plugin>
@@ -30,13 +26,69 @@
         </xacro:unless>
       </hardware>
-      <joint name="${prefix}left_wheel_joint">
-        <command_interface name="velocity"/>
-        <state_interface name="position"/>
+      <joint name="${prefix}joint1">
+        <command_interface name="position">     <!-- Add/Remove interfaces as needed -->
+          <param name="min">-1</param>
+          <param name="max">1</param>
+        </command_interface>
+        <state_interface name="position">
+          <param name="initial_value">0.0</param>
+        </state_interface>
         <state_interface name="velocity"/>
+        <state_interface name="acceleration"/>
       </joint>
-      <joint name="${prefix}right_wheel_joint">
-        <command_interface name="velocity"/>
-        <state_interface name="position"/>
+      <joint name="${prefix}joint2">
+        <command_interface name="position">     <!-- Add/Remove interfaces as needed -->
+          <param name="min">-1</param>
+          <param name="max">1</param>
+        </command_interface>
+        <state_interface name="position">
+          <param name="initial_value">0.0</param>
+        </state_interface>
         <state_interface name="velocity"/>
+        <state_interface name="acceleration"/>
+      </joint>
+      <joint name="${prefix}joint3">
+        <command_interface name="position">     <!-- Add/Remove interfaces as needed -->
+          <param name="min">-1</param>
+          <param name="max">1</param>
+        </command_interface>
+        <state_interface name="position">
+          <param name="initial_value">0.0</param>
+        </state_interface>
+        <state_interface name="velocity"/>
+        <state_interface name="acceleration"/>
+      </joint>
+      <joint name="${prefix}joint4">
+        <command_interface name="position">     <!-- Add/Remove interfaces as needed -->
+          <param name="min">-1</param>
+          <param name="max">1</param>
+        </command_interface>
+        <state_interface name="position">
+          <param name="initial_value">0.0</param>
+        </state_interface>
+        <state_interface name="velocity"/>
+        <state_interface name="acceleration"/>
+      </joint>
+      <joint name="${prefix}joint5">
+        <command_interface name="position">     <!-- Add/Remove interfaces as needed -->
+          <param name="min">-1</param>
+          <param name="max">1</param>
+        </command_interface>
+        <state_interface name="position">
+          <param name="initial_value">0.0</param>
+        </state_interface>
+        <state_interface name="velocity"/>
+        <state_interface name="acceleration"/>
+      </joint>
+      <joint name="${prefix}joint6">
+        <command_interface name="position">     <!-- Add/Remove interfaces as needed -->
+          <param name="min">-1</param>
+          <param name="max">1</param>
+        </command_interface>
+        <state_interface name="position">
+          <param name="initial_value">0.0</param>
+        </state_interface>
+        <state_interface name="velocity"/>
+        <state_interface name="acceleration"/>
       </joint>
       <sensor name="tcp_fts_sensor">            <!-- Remove/change sensors as needed -->

File: plastic_description/urdf/plastic/plastic_macro.xacro (robot description, xacro)
@@ -1,16 +1,5 @@
 <?xml version="1.0" encoding="UTF-8"?>
 <robot xmlns:xacro="http://wiki.ros.org/xacro">
-  <xacro:property name="base_width" value="0.1"/>
-  <xacro:property name="base_length" value="0.175"/>
-  <xacro:property name="base_height" value="0.088"/>
-  <xacro:property name="base_xoff" value="0.05"/>
-  <xacro:property name="wheel_radius" value="0.033"/>
-  <xacro:property name="wheel_width" value="0.025"/>
-  <xacro:property name="wheel_ygap" value="0.0125"/>
-  <xacro:property name="axle_zoff" value="0.01"/>
-  <xacro:property name="caster_xoff" value="0.02"/>
-  <xacro:property name="laser_radius" value="0.035"/>
-  <xacro:property name="laser_height" value="0.055"/>
-  <xacro:property name="laser_zoff" value="0.0175"/>
+  <xacro:include filename="$(find plastic_description)/urdf/common.xacro" />
   <xacro:macro name="plastic" params="prefix parent *origin">
     <!-- LINKS -->
@@ -21,15 +10,38 @@
       <xacro:default_inertial/>
       <visual>
-        <geometry>
-          <box size="${base_length} ${base_width} ${base_height}"/>
-        </geometry>
-        <origin xyz="${-(base_xoff)} 0.0 0.0" rpy="0 0 0"/>
-        <material name="Cyan">
-          <color rgba="0 1.0 1.0 1.0"/>
-        </material>
-      </visual>
+        <origin xyz="0 0 0" rpy="0 0 0" />
+        <geometry>
+          <cylinder length="0.3" radius="0.3" />
+<!--           <mesh filename="package://plastic_description/meshes/plastic/visual/base_link.dae" /> -->
+        </geometry>
+      </visual>
+      <collision>
+        <origin xyz="0 0 0" rpy="0 0 0" />
+        <geometry>
+          <cylinder length="0.3" radius="0.3" />
+<!--           <mesh filename="package://plastic_description/meshes/plastic/collision/base_link.stl" /> -->
+        </geometry>
+      </collision>
     </link>
     <!-- link 1 -->
-    <link name="${prefix}base_footprint" />
+    <link name="${prefix}link1">
+      <!-- Default inertial for Gazebo/Ingnition - copy and edit block from 'common.xacro'
+           to get more realistic behaviour-->
+      <xacro:default_inertial/>
+      <visual>
+        <origin xyz="0 0 0" rpy="0 0 0" />
+        <geometry>
+          <cylinder length="0.3" radius="0.15" />
+<!--           <mesh filename="package://plastic_description/meshes/plastic/visual/link1.dae" /> -->
+        </geometry>
+      </visual>
+      <collision>
+        <origin xyz="0 0 0" rpy="0 0 0" />
+        <geometry>
+          <cylinder length="0.3" radius="0.15" />
+<!--           <mesh filename="package://plastic_description/meshes/plastic/collision/link1.stl" /> -->
+        </geometry>
+      </collision>
+    </link>
     <!-- link 2 -->
     <link name="${prefix}link2">
@@ -135,4 +147,13 @@
     <link name="${prefix}tool0" />
     <!-- tool link -->
+<!-- START Delete if not needed -->
+    <!-- Standard frames for industrial robots. Also useful for manipulators.
+         (ROS-I specs - https://wiki.ros.org/Industrial/Tutorials/WorkingWithRosIndustrialRobotSupportPackages#Standardised_links_.2F_frames)-->
+    <!-- This frame should correspond to the BASE coordinate system of robot's controller.) -->
+    <link name="${prefix}base" />
+    <!-- Frame for mounting EEF models to a manipulator. x+ axis points forward (REP 103). -->
+    <link name="${prefix}flange" />
+<!-- END Delete if not needed  -->
+    <!-- END LINKS -->
     <!-- JOINTS -->
     <!-- base_joint fixes base_link to the environment -->
